File: SignalSlinger/KiCad/SignalSlinger/Misc.kicad_sch (KiCad schematic)
At the start: 13 parts

Commit message: Updates
Schematic and PCB updates
Parts:
- added HDWR413: (no value), symbol Graphic:Logo_Open_Hardware_Large
Other:
- note added: "Core Product"
- note added: "FTDI Support"
- note added: "Internal Battery Support"
- title: (none) -> SignalSlinger Design
- moved on the sheet: BT401

Commit message: Schematic Debug
Fixed misplaced varistor
Parts:
- HDWR413: value (none) -> FTDI Adapter PCB
Changed lines of the file:
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@@
       (effects (font (size 1.27 1.27)) hide)
     )
-    (property "Value" "" (id 1) (at 153.67 143.51 0))
+    (property "Value" "FTDI Adapter PCB" (id 1) (at 153.67 143.51 0))
     (property "Footprint" "" (id 2) (at 153.67 133.35 0)
       (effects (font (size 1.27 1.27)) hide)
