File: SignalSlinger/KiCad/SignalSlinger/PowerSupply.kicad_sch (KiCad schematic)
At the start: 29 parts, among them J201 Barrel_Jack_Switch, J202 Conn_01x03, U201 LP2985-3.3, U202 LP2985-3.3, U203 TPS63060

Commit message: Updates
Schematic and PCB updates
Parts:
- added R205: 105k, Resistor_SMD:R_0805_2012Metric, symbol Device:R_Small_US
Connections:
- net B/B_PS_Enable: now also R205.1
- net GND: now also R205.2
Other:
- title: (none) -> SignalSlinger Design
- moved on the sheet: C204, C205, C207, C208, J201, J202, L201

Commit message: PCB Development
First cut at traces
Parts:
- BT201: footprint Connector_Wire:SolderWire-2.5sqmm_1x02_P7.2mm_D2.4mm_OD3.6mm -> Connector_Wire:SolderWire-0.5sqmm_1x02_P4.6mm_D0.9mm_OD2.1mm
- C201, C202, C203, C205, C206, C207, C209, C210: footprint Capacitor_SMD:C_0805_2012Metric_Pad1.18x1.45mm_HandSolder -> Capacitor_SMD:C_0805_2012Metric
Connections:
- net +BATT: now also BT201.2 (+); no longer BT201.1 (+)
- net GND: now also BT201.1 (-); no longer BT201.2 (-)
Changed lines of the file:
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@@
       (effects (font (size 1.27 1.27)) (justify left))
     )
-    (property "Footprint" "Connector_Wire:SolderWire-2.5sqmm_1x02_P7.2mm_D2.4mm_OD3.6mm" (id 2) (at 55.88 175.006 90)
+    (property "Footprint" "Connector_Wire:SolderWire-0.5sqmm_1x02_P4.6mm_D0.9mm_OD2.1mm" (id 2) (at 55.88 175.006 90)
       (effects (font (size 1.27 1.27)) hide)
     )
@@
     (property "Reference" "C203" (id 0) (at 92.71 132.08 90))
     (property "Value" "10uF" (id 1) (at 91.44 137.16 90))
-    (property "Footprint" "Capacitor_SMD:C_0805_2012Metric_Pad1.18x1.45mm_HandSolder" (id 2) (at 86.36 134.62 0)
+    (property "Footprint" "Capacitor_SMD:C_0805_2012Metric" (id 2) (at 86.36 134.62 0)
       (effects (font (size 1.27 1.27)) hide)
     )
@@
     (property "Reference" "C206" (id 0) (at 115.57 124.46 90))
     (property "Value" "10uF" (id 1) (at 110.49 120.65 90))
-    (property "Footprint" "Capacitor_SMD:C_0805_2012Metric_Pad1.18x1.45mm_HandSolder" (id 2) (at 113.03 125.73 0)
+    (property "Footprint" "Capacitor_SMD:C_0805_2012Metric" (id 2) (at 113.03 125.73 0)
       (effects (font (size 1.27 1.27)) hide)
     )
@@
     (property "Reference" "C205" (id 0) (at 90.17 85.09 90))
     (property "Value" "10uF" (id 1) (at 95.25 86.36 90))
-    (property "Footprint" "Capacitor_SMD:C_0805_2012Metric_Pad1.18x1.45mm_HandSolder" (id 2) (at 92.71 82.55 0)
+    (property "Footprint" "Capacitor_SMD:C_0805_2012Metric" (id 2) (at 92.71 82.55 0)
       (effects (font (size 1.27 1.27)) hide)
     )
@@
     (property "Reference" "C201" (id 0) (at 50.8 134.62 90))
     (property "Value" "10uF" (id 1) (at 49.53 139.7 90))
-    (property "Footprint" "Capacitor_SMD:C_0805_2012Metric_Pad1.18x1.45mm_HandSolder" (id 2) (at 53.34 137.16 0)
+    (property "Footprint" "Capacitor_SMD:C_0805_2012Metric" (id 2) (at 53.34 137.16 0)
       (effects (font (size 1.27 1.27)) hide)
     )
@@
       (effects (font (size 1.27 1.27)) (justify left))
     )
-    (property "Footprint" "Capacitor_SMD:C_0805_2012Metric_Pad1.18x1.45mm_HandSolder" (id 2) (at 138.43 142.24 0)
+    (property "Footprint" "Capacitor_SMD:C_0805_2012Metric" (id 2) (at 138.43 142.24 0)
       (effects (font (size 1.27 1.27)) hide)
     )
@@
     (property "Reference" "C210" (id 0) (at 144.78 133.35 90))
     (property "Value" "10uF" (id 1) (at 146.05 138.43 90))
-    (property "Footprint" "Capacitor_SMD:C_0805_2012Metric_Pad1.18x1.45mm_HandSolder" (id 2) (at 142.24 135.89 0)
+    (property "Footprint" "Capacitor_SMD:C_0805_2012Metric" (id 2) (at 142.24 135.89 0)
       (effects (font (size 1.27 1.27)) hide)
     )
@@
       (effects (font (size 1.27 1.27)) (justify left))
     )
-    (property "Footprint" "Capacitor_SMD:C_0805_2012Metric_Pad1.18x1.45mm_HandSolder" (id 2) (at 57.15 143.51 0)
+    (property "Footprint" "Capacitor_SMD:C_0805_2012Metric" (id 2) (at 57.15 143.51 0)
       (effects (font (size 1.27 1.27)) hide)
     )
@@
     (property "Reference" "C207" (id 0) (at 96.52 85.09 90))
     (property "Value" "10uF" (id 1) (at 101.6 86.36 90))
-    (property "Footprint" "Capacitor_SMD:C_0805_2012Metric_Pad1.18x1.45mm_HandSolder" (id 2) (at 99.06 82.55 0)
-      (effects (font (size 1.27 1.27)) hide)
-    )
+    (property "Footprint" "Capacitor_SMD:C_0805_2012Metric" (id 2) (at 99.06 82.55 0)
+      (effects (font (size 1.27 1.27)) hide)
+    )

Commit message: BOM
Updates to BOM parts
Parts:
- C201, C203, C205, C206, C207, C210: value 10uF -> (none); footprint Capacitor_SMD:C_0805_2012Metric -> (none); Digi-Key Part No. 1276-1764-1-ND -> 445-14418-1-ND; LCSC Part Number (none) -> C3843628; Link (none) -> https://www.digikey.com/short/p8qdn4mp; Manufacturer Samsung Electro-Mechanics -> TDK Corporation; Manufacturer PN CL21B106KPQNNNE -> C2012X5R1V106K125AC
- C202, C209: value 10nF -> (none); footprint Capacitor_SMD:C_0805_2012Metric -> (none); Digi-Key Part No. 1276-1015-1-ND -> 399-C0805C103J5GEC7800CT-ND; LCSC Part Number (none) -> C3887673; Link (none) -> https://www.digikey.com/short/qd893213; Manufacturer Samsung Electro-Mechanics -> KEMET; Manufacturer PN CL21B103KBANNNC -> C0805C103J5GEC7800
- C204: value 470nF -> (none); footprint Capacitor_SMD:C_0805_2012Metric -> (none); Link <a href="https://www.digikey.com/products/en?keywords=478-9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 -> https://www.digikey.com/products/en?keywords=478-9924-1-ND
- C208: value 100nF -> (none); footprint Capacitor_SMD:C_0805_2012Metric -> (none); LCSC Part Number (none) -> C29926; Link (none) -> https://www.digikey.com/short/q2f22qnq
- C211: value 10pF -> (none); footprint Capacitor_SMD:C_0805_2012Metric -> (none); LCSC Part Number (none) -> C157608
- C212: value 1uF -> (none); footprint Capacitor_SMD:C_0805_2012Metric -> (none); LCSC Part Number (none) -> C28323
- C213, C214, C215: value 22uF -> (none); footprint Capacitor_SMD:C_1210_3225Metric -> (none); Link <a href="https://www.digikey.com/products/en?keywords=1276-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 -> https://www.digikey.com/products/en?keywords=1276-3373-1-ND
- D201: value BAT54C -> (none); footprint Package_TO_SOT_SMD:SC-59 -> (none); LCSC Part Number (none) -> C37704
- L201: value choke -> (none); footprint Inductor_SMD:L_Wuerth_WE-LQS -> (none); LCSC Part Number (none) -> C2041406
- R201, R203: value 105k -> (none); footprint Resistor_SMD:R_0805_2012Metric -> (none); LCSC Part Number (none) -> C273877
- R202, R204: value 1M -> (none); footprint Resistor_SMD:R_0805_2012Metric -> (none); LCSC Part Number (none) -> C4198744
- U201, U202: value LP2985-3.3 -> (none); footprint Package_TO_SOT_SMD:SOT-23-5 -> (none); LCSC Part Number (none) -> C89826; Link (none) -> https://www.digikey.com/short/vr2m3rjp
- U203: value TPS63060 -> (none); footprint Package_SON:Texas_S-PWSON-N10_ThermalVias -> (none); LCSC Part Number (none) -> C2070911

Commit message: Development
o Added polarity protection diode
o Tweaks to PCB
Parts:
- added D202: (no value), symbol Device:D_Schottky_Filled
- C201, C203, C205, C206, C207, C210: value (none) -> 10uF; footprint (none) -> Capacitor_SMD:C_0805_2012Metric
- C202, C209: value (none) -> 10nF; footprint (none) -> Capacitor_SMD:C_0805_2012Metric
- C204: value (none) -> 470nF; footprint (none) -> Capacitor_SMD:C_0805_2012Metric
- C208: value (none) -> 100nF; footprint (none) -> Capacitor_SMD:C_0805_2012Metric
- C211: value (none) -> 10pF; footprint (none) -> Capacitor_SMD:C_0805_2012Metric
- C212: value (none) -> 1uF; footprint (none) -> Capacitor_SMD:C_0805_2012Metric
- C213, C214, C215: value (none) -> 22uF; footprint (none) -> Capacitor_SMD:C_1210_3225Metric
- D201: value (none) -> BAT54C; footprint (none) -> Package_TO_SOT_SMD:SC-59
- L201: value (none) -> 2.2uH; footprint (none) -> Inductor_SMD:L_Wuerth_WE-LQS
- R201, R203: value (none) -> 105k; footprint (none) -> Resistor_SMD:R_0805_2012Metric
- R202, R204: value (none) -> 1M; footprint (none) -> Resistor_SMD:R_0805_2012Metric
- U201, U202: value (none) -> LP2985-3.3; footprint (none) -> Package_TO_SOT_SMD:SOT-23-5
- U203: value (none) -> TPS63060; footprint (none) -> Package_SON:Texas_S-PWSON-N10_ThermalVias
Connections:
- net +BATT: now also BT201.1 (+); no longer BT201.2 (+)
- net GND: now also BT201.2 (-); no longer BT201.1 (-)
- net at L201.1: now also D202.1 (K); no longer J201.1
- new net: D202.2 (A), J201.1
Other:
- moved on the sheet: J201

Commit message: Minor Edits
Schematic and PCB tweaks
Parts:
- D202: value (none) -> B330A Schottky Diode; footprint (none) -> Diode_SMD:D_SMA
Changed lines of the file:
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@@
     (in_bom yes) (on_board yes) (fields_autoplaced)
     (property "Reference" "D202" (id 0) (at 57.4675 53.4472 0))
-    (property "Value" "" (id 1) (at 57.4675 53.4471 0)
+    (property "Value" "B330A Schottky Diode" (id 1) (at 57.4675 53.4471 0)
       (effects (font (size 1.27 1.27)) hide)
     )
-    (property "Footprint" "" (id 2) (at 57.15 55.88 0)
+    (property "Footprint" "Diode_SMD:D_SMA" (id 2) (at 57.15 55.88 0)
       (effects (font (size 1.27 1.27)) hide)
     )
