File: SignalSlinger/KiCad/SignalSlinger/RF_Filters.kicad_sch (KiCad schematic)
At the start: 13 parts, among them J301 To Antenna, J302 Conn_01x03

Commit message: Updates
Schematic and PCB updates
Other:
- title: (none) -> SignalSlinger Design
Changed lines of the file:
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@@
 (kicad_sch (version 20211123) (generator eeschema)
   (paper "A4")
+  (title_block
+    (title "SignalSlinger Design")
+    (date "2023-06-20")
+    (rev "1.0")
+  )
   (junction (at 165.1 83.82) (diameter 0) (color 0 0 0 0)
   )

Commit message: BOM
Updates to BOM parts
Parts:
- C301: value 470nF -> (none); footprint Capacitor_SMD:C_0805_2012Metric -> (none); Link <a href="https://www.digikey.com/products/en?keywords=478-9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 -> https://www.digikey.com/products/en?keywords=478-9924-1-ND
- C302, C305: value 1100pF -> (none); footprint Capacitor_THT:C_Rect_L7.0mm_W2.5mm_P5.00mm -> (none); Link <a href="https://www.digikey.com/products/en?keywords=399-1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 -> https://www.digikey.com/products/en?keywords=399-14552-1-ND
- C303: value 1800pF -> (none); footprint Capacitor_THT:C_Rect_L7.0mm_W2.5mm_P5.00mm -> (none); Link <a href="https://www.digikey.com/products/en?keywords=445-5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 -> https://www.digikey.com/products/en?keywords=445-5752-1-ND
- C304: value 91pF -> (none); footprint Capacitor_THT:C_Rect_L7.0mm_W2.5mm_P5.00mm -> (none); Link <a href="https://www.digikey.com/products/en?keywords=478-1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 -> https://www.digikey.com/products/en?keywords=478-10247-1-ND
- L301, L302: value 2.7uH -> (none); footprint Inductors:Toroid_T-60_2TH -> (none); Link <a href="http://www.amidoncorp.com/t60-2/">Link</a> -> http://www.amidoncorp.com/t60-2/
Changed lines of the file:
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@@
       (effects (font (size 1.27 1.27)) (justify left))
     )
-    (property "Value" "1800pF" (id 1) (at 142.24 91.44 0)
-      (effects (font (size 1.27 1.27)) (justify left))
-    )
-    (property "Footprint" "Capacitor_THT:C_Rect_L7.0mm_W2.5mm_P5.00mm" (id 2) (at 134.62 88.9 0)
+    (property "Value" "" (id 1) (at 142.24 91.44 0)
+      (effects (font (size 1.27 1.27)) (justify left))
+    )
+    (property "Footprint" "" (id 2) (at 134.62 88.9 0)
       (effects (font (size 1.27 1.27)) hide)
     )
@@
       (effects (font (size 1.27 1.27)) hide)
     )
-    (property "Link" "<a href=\"https://www.digikey.com/products/en?keywords=445-5752-1-ND\">Link</a>" (id 5) (at 134.62 88.9 0)
+    (property "Link" "https://www.digikey.com/products/en?keywords=445-5752-1-ND" (id 5) (at 134.62 88.9 0)
       (effects (font (size 1.524 1.524)) hide)
     )
@@
       (effects (font (size 1.27 1.27)) (justify left))
     )
-    (property "Value" "1100pF" (id 1) (at 160.274 90.932 0)
-      (effects (font (size 1.27 1.27)) (justify left))
-    )
-    (property "Footprint" "Capacitor_THT:C_Rect_L7.0mm_W2.5mm_P5.00mm" (id 2) (at 160.02 88.9 0)
+    (property "Value" "" (id 1) (at 160.274 90.932 0)
+      (effects (font (size 1.27 1.27)) (justify left))
+    )
+    (property "Footprint" "" (id 2) (at 160.02 88.9 0)
       (effects (font (size 1.27 1.27)) hide)
     )
@@
       (effects (font (size 1.27 1.27)) hide)
     )
-    (property "Link" "<a href=\"https://www.digikey.com/products/en?keywords=399-14552-1-ND\">Link</a>" (id 5) (at 160.02 88.9 0)
+    (property "Link" "https://www.digikey.com/products/en?keywords=399-14552-1-ND" (id 5) (at 160.02 88.9 0)
       (effects (font (size 1.524 1.524)) hide)
     )
@@
       (effects (font (size 1.27 1.27)) (justify left))
     )
-    (property "Value" "1100pF" (id 1) (at 117.094 90.932 0)
-      (effects (font (size 1.27 1.27)) (justify left))
-    )
-    (property "Footprint" "Capacitor_THT:C_Rect_L7.0mm_W2.5mm_P5.00mm" (id 2) (at 116.84 88.9 0)
+    (property "Value" "" (id 1) (at 117.094 90.932 0)
+      (effects (font (size 1.27 1.27)) (justify left))
+    )
+    (property "Footprint" "" (id 2) (at 116.84 88.9 0)
       (effects (font (size 1.27 1.27)) hide)
     )
@@
       (effects (font (size 1.27 1.27)) hide)
     )
-    (property "Link" "<a href=\"https://www.digikey.com/products/en?keywords=399-14552-1-ND\">Link</a>" (id 5) (at 116.84 88.9 0)
+    (property "Link" "https://www.digikey.com/products/en?keywords=399-14552-1-ND" (id 5) (at 116.84 88.9 0)
       (effects (font (size 1.524 1.524)) hide)
     )
@@
     (in_bom yes) (on_board yes)
     (property "Reference" "L302" (id 0) (at 151.13 81.28 0))
-    (property "Value" "2.7uH" (id 1) (at 151.13 85.09 0))
-    (property "Footprint" "Inductors:Toroid_T-60_2TH" (id 2) (at 151.13 83.82 0)
+    (property "Value" "" (id 1) (at 151.13 85.09 0))
+    (property "Footprint" "" (id 2) (at 151.13 83.82 0)
       (effects (font (size 1.27 1.27)) hide)
     )
@@
       (effects (font (size 1.27 1.27)) hide)
     )
-    (property "Link" "<a href=\"http://www.amidoncorp.com/t60-2/\">Link</a>" (id 5) (at 151.13 83.82 0)
+    (property "Link" "http://www.amidoncorp.com/t60-2/" (id 5) (at 151.13 83.82 0)
       (effects (font (size 1.524 1.524)) hide)
     )
@@
     (in_bom yes) (on_board yes)
     (property "Reference" "L301" (id 0) (at 125.73 81.28 0))
-    (property "Value" "2.7uH" (id 1) (at 125.73 85.09 0))
-    (property "Footprint" "Inductors:Toroid_T-60_2TH" (id 2) (at 125.73 83.82 0)
+    (property "Value" "" (id 1) (at 125.73 85.09 0))
+    (property "Footprint" "" (id 2) (at 125.73 83.82 0)
       (effects (font (size 1.27 1.27)) hide)
     )
@@
       (effects (font (size 1.27 1.27)) hide)
     )
-    (property "Link" "<a href=\"http://www.amidoncorp.com/t60-2/\">Link</a>" (id 5) (at 125.73 83.82 0)
+    (property "Link" "http://www.amidoncorp.com/t60-2/" (id 5) (at 125.73 83.82 0)
       (effects (font (size 1.524 1.524)) hide)
     )
@@
       (effects (font (size 1.27 1.27)) (justify left))
     )
-    (property "Value" "470nF" (id 1) (at 111.76 87.63 90)
-      (effects (font (size 1.27 1.27)) (justify left))
-    )
-    (property "Footprint" "Capacitor_SMD:C_0805_2012Metric" (id 2) (at 109.22 83.82 0)
+    (property "Value" "" (id 1) (at 111.76 87.63 90)
+      (effects (font (size 1.27 1.27)) (justify left))
+    )
+    (property "Footprint" "" (id 2) (at 109.22 83.82 0)
       (effects (font (size 1.27 1.27)) hide)
     )
@@
       (effects (font (size 1.27 1.27)) hide)
     )
-    (property "Link" "<a href=\"https://www.digikey.com/products/en?keywords=478-9924-1-ND\">Link</a>" (id 5) (at 109.22 83.82 0)
+    (property "Link" "https://www.digikey.com/products/en?keywords=478-9924-1-ND" (id 5) (at 109.22 83.82 0)
       (effects (font (size 1.524 1.524)) hide)
     )
@@
       (effects (font (size 1.27 1.27)) (justify left))
     )
-    (property "Value" "91pF" (id 1) (at 148.59 78.74 90)
-      (effects (font (size 1.27 1.27)) (justify left))
-    )
-    (property "Footprint" "Capacitor_THT:C_Rect_L7.0mm_W2.5mm_P5.00mm" (id 2) (at 151.13 76.2 0)
+    (property "Value" "" (id 1) (at 148.59 78.74 90)
+      (effects (font (size 1.27 1.27)) (justify left))
+    )
+    (property "Footprint" "" (id 2) (at 151.13 76.2 0)
       (effects (font (size 1.27 1.27)) hide)
     )
@@
       (effects (font (size 1.27 1.27)) hide)
     )
-    (property "Link" "<a href=\"https://www.digikey.com/products/en?keywords=478-10247-1-ND\">Link</a>" (id 5) (at 151.13 76.2 0)
-      (effects (font (size 1.524 1.524)) hide)
-    )
+    (property "Link" "https://www.digikey.com/products/en?keywords=478-10247-1-ND" (id 5) (at 151.13 76.2 0)
+      (effects (font (size 1.524 1.524)) hide)
+    )

Commit message: Development
o Added polarity protection diode
o Tweaks to PCB
Parts:
- C301: value (none) -> 470nF; footprint (none) -> Capacitor_SMD:C_0805_2012Metric
- C302, C305: value (none) -> 1100pF; footprint (none) -> Capacitor_THT:C_Rect_L7.0mm_W2.5mm_P5.00mm
- C303: value (none) -> 1800pF; footprint (none) -> Capacitor_THT:C_Rect_L7.0mm_W2.5mm_P5.00mm
- C304: value (none) -> 91pF; footprint (none) -> Capacitor_THT:C_Rect_L7.0mm_W2.5mm_P5.00mm
- L301, L302: value (none) -> 2.7uH; footprint (none) -> Inductors:Toroid_T-60_2TH
Changed lines of the file:
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@@
       (effects (font (size 1.27 1.27)) (justify left))
     )
-    (property "Value" "" (id 1) (at 142.24 91.44 0)
-      (effects (font (size 1.27 1.27)) (justify left))
-    )
-    (property "Footprint" "" (id 2) (at 134.62 88.9 0)
+    (property "Value" "1800pF" (id 1) (at 142.24 91.44 0)
+      (effects (font (size 1.27 1.27)) (justify left))
+    )
+    (property "Footprint" "Capacitor_THT:C_Rect_L7.0mm_W2.5mm_P5.00mm" (id 2) (at 134.62 88.9 0)
       (effects (font (size 1.27 1.27)) hide)
     )
@@
       (effects (font (size 1.27 1.27)) (justify left))
     )
-    (property "Value" "" (id 1) (at 160.274 90.932 0)
-      (effects (font (size 1.27 1.27)) (justify left))
-    )
-    (property "Footprint" "" (id 2) (at 160.02 88.9 0)
+    (property "Value" "1100pF" (id 1) (at 160.274 90.932 0)
+      (effects (font (size 1.27 1.27)) (justify left))
+    )
+    (property "Footprint" "Capacitor_THT:C_Rect_L7.0mm_W2.5mm_P5.00mm" (id 2) (at 160.02 88.9 0)
       (effects (font (size 1.27 1.27)) hide)
     )
@@
       (effects (font (size 1.27 1.27)) (justify left))
     )
-    (property "Value" "" (id 1) (at 117.094 90.932 0)
-      (effects (font (size 1.27 1.27)) (justify left))
-    )
-    (property "Footprint" "" (id 2) (at 116.84 88.9 0)
+    (property "Value" "1100pF" (id 1) (at 117.094 90.932 0)
+      (effects (font (size 1.27 1.27)) (justify left))
+    )
+    (property "Footprint" "Capacitor_THT:C_Rect_L7.0mm_W2.5mm_P5.00mm" (id 2) (at 116.84 88.9 0)
       (effects (font (size 1.27 1.27)) hide)
     )
@@
     (in_bom yes) (on_board yes)
     (property "Reference" "L302" (id 0) (at 151.13 81.28 0))
-    (property "Value" "" (id 1) (at 151.13 85.09 0))
-    (property "Footprint" "" (id 2) (at 151.13 83.82 0)
+    (property "Value" "2.7uH" (id 1) (at 151.13 85.09 0))
+    (property "Footprint" "Inductors:Toroid_T-60_2TH" (id 2) (at 151.13 83.82 0)
       (effects (font (size 1.27 1.27)) hide)
     )
@@
     (in_bom yes) (on_board yes)
     (property "Reference" "L301" (id 0) (at 125.73 81.28 0))
-    (property "Value" "" (id 1) (at 125.73 85.09 0))
-    (property "Footprint" "" (id 2) (at 125.73 83.82 0)
+    (property "Value" "2.7uH" (id 1) (at 125.73 85.09 0))
+    (property "Footprint" "Inductors:Toroid_T-60_2TH" (id 2) (at 125.73 83.82 0)
       (effects (font (size 1.27 1.27)) hide)
     )
@@
       (effects (font (size 1.27 1.27)) (justify left))
     )
-    (property "Value" "" (id 1) (at 111.76 87.63 90)
-      (effects (font (size 1.27 1.27)) (justify left))
-    )
-    (property "Footprint" "" (id 2) (at 109.22 83.82 0)
+    (property "Value" "470nF" (id 1) (at 111.76 87.63 90)
+      (effects (font (size 1.27 1.27)) (justify left))
+    )
+    (property "Footprint" "Capacitor_SMD:C_0805_2012Metric" (id 2) (at 109.22 83.82 0)
       (effects (font (size 1.27 1.27)) hide)
     )
@@
       (effects (font (size 1.27 1.27)) (justify left))
     )
-    (property "Value" "" (id 1) (at 148.59 78.74 90)
-      (effects (font (size 1.27 1.27)) (justify left))
-    )
-    (property "Footprint" "" (id 2) (at 151.13 76.2 0)
-      (effects (font (size 1.27 1.27)) hide)
-    )
+    (property "Value" "91pF" (id 1) (at 148.59 78.74 90)
+      (effects (font (size 1.27 1.27)) (justify left))
+    )
+    (property "Footprint" "Capacitor_THT:C_Rect_L7.0mm_W2.5mm_P5.00mm" (id 2) (at 151.13 76.2 0)
+      (effects (font (size 1.27 1.27)) hide)
+    )

Commit message: Minor Edits
Schematic and PCB tweaks
Parts:
- J301: value To Antenna -> (none); footprint Connector_Coaxial:BNC_TEConnectivity_1478035_Horizontal -> (none)
Changed lines of the file:
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@@
       (effects (font (size 1.27 1.27)) (justify left))
     )
-    (property "Value" "To Antenna" (id 1) (at 180.3401 85.8154 0)
+    (property "Value" "" (id 1) (at 180.3401 85.8154 0)
       (effects (font (size 1.27 1.27)) (justify left))
     )
-    (property "Footprint" "Connector_Coaxial:BNC_TEConnectivity_1478035_Horizontal" (id 2) (at 177.8 83.82 0)
+    (property "Footprint" "" (id 2) (at 177.8 83.82 0)
       (effects (font (size 1.27 1.27)) hide)
     )
