File: SignalSlinger/KiCad/SignalSlinger/SignalSlinger.kicad_sch (KiCad schematic)
At the start: 65 parts, among them J101 Conn_01x02, J103 Conn_01x02, J104 Conn_01x02, J105 Conn_01x02, J106 Conn_01x02, J108 Conn_01x02, J109 Conn_01x03, J110 Conn_01x02, J111 Conn_01x03, J112 External Power Source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

Commit message: Development
o Added polarity protection diode
o Tweaks to PCB
Parts:
- C101, C104, C105, C107: value (none) -> 100nF; footprint (none) -> Capacitor_SMD:C_0805_2012Metric
- C102, C103, C106, C108, C112, C113, C114: value (none) -> 470nF; footprint (none) -> Capacitor_SMD:C_0805_2012Metric
- C109, C116: value (none) -> 10uF; footprint (none) -> Capacitor_SMD:C_0805_2012Metric
- C110: value (none) -> 22uF; footprint (none) -> Capacitor_SMD:C_1210_3225Metric
- C111: value (none) -> 47uF low ESR; footprint (none) -> Capacitors:C_2917
- C115: value (none) -> C_Trim_Small; footprint (none) -> Capacitors:MURATA-TZC3
- D101, D102: value (none) -> 1N914WT; footprint (none) -> Diode_SMD:D_SOD-523
- D103: value (none) -> Red LED; footprint (none) -> LED_SMD:LED_0805_2012Metric
- D104: value (none) -> Green LED; footprint (none) -> LED_SMD:LED_APDA1806SECK
- D105, D106, D108, D109, D110: value (none) -> ESD9B5.0ST5G_1; footprint (none) -> Diode_SMD:D_0603_1608Metric
- D107: value (none) -> MBRD10100CT; footprint (none) -> Package_TO_SOT_SMD:TO-252-2
- J107: value (none) -> DB9 Female; footprint (none) -> Connector_Dsub:DSUB-9_Female_EdgeMount_P2.77mm
- L101: value (none) -> 9T #24 Bifilar T50-43; footprint (none) -> Inductors:Toroid_T-50A_TH_BF_CT
- L102: value (none) -> INDUCTOR_tapped; footprint (none) -> Inductors:Toroid_T-50A_TH_BF_CT_Vertical
- P101: value (none) -> ISP/PDI; footprint (none) -> Connector_PinHeader_2.54mm:PinHeader_2x03_P2.54mm_Vertical_SMD
- Q101: value (none) -> BSS84W-7-F; footprint (none) -> Package_TO_SOT_SMD:SOT-323_SC-70
- Q102: value (none) -> BSS138W-7-F; footprint (none) -> Package_TO_SOT_SMD:SOT-323_SC-70
- Q103: value (none) -> IRF610; footprint (none) -> TO_SOT_Packages:TO-220_Neutral123_Vertical_LargePads
- R101: value (none) -> 105k; footprint (none) -> Resistor_SMD:R_0805_2012Metric
- R102: value (none) -> 162k; footprint (none) -> Resistor_SMD:R_0805_2012Metric
- R103: value (none) -> 12.4k; footprint (none) -> Resistor_SMD:R_0805_2012Metric
- R104, R105: value (none) -> 1k; footprint (none) -> Resistor_SMD:R_0805_2012Metric
- R106: value (none) -> 47k; footprint (none) -> Resistor_SMD:R_0805_2012Metric
- R107, R108: value (none) -> 10k; footprint (none) -> Capacitor_SMD:C_0805_2012Metric
- U101: value (none) -> AVR128DA28; footprint (none) -> Package_SO:SOIC-28W_7.5x17.9mm_P1.27mm
- U102: value (none) -> SI5351; footprint (none) -> Package_SO:MSOP-10_3x3mm_P0.5mm
- U104: value (none) -> LM5134; footprint (none) -> Package_TO_SOT_SMD:SOT-23-6-LM5134
- X101: value (none) -> SIT1566AC TCO; footprint (none) -> Oscillator:Oscillator_SMD_SiTime_SIT1566AC-4Pin_BGA
- X102: value (none) -> 25 MHz; footprint (none) -> Crystal:Crystal_SMD_TXETCLSANF-4Pin
