File: KiCad/SignalSlinger/SignalSlinger_original_L201.kicad_pcb (KiCad board)
At the start: 2 copper layers, 92.1 x 59.1 mm, 106 parts, among them J101 Conn_01x02, J102 Conn_01x03, J103 Conn_01x02, J104 Conn_01x02, J105 Conn_01x04, J106 Conn_01x02, J107 DB9 Female, J108 Conn_01x02, J109 Conn_01x03, J201 Barrel_Jack_Switch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

Commit message: KiCad Updates
Updated Gerbers and schematic
Parts:
- removed J105: Conn_01x04, Connector_PinHeader_2.54mm:PinHeader_1x04_P2.54mm_Vertical
- L201: footprint Inductor_SMD:WPN4020H2R2MT -> Inductor_SMD:L_Wuerth_WE-LQS
Connections:
- R205 pad 1: GND -> B/B_PS_Enable
- R205 pad 2: B/B_PS_Enable -> GND
Routing:
- net Straightkey: track 27.8 -> 17.1 mm, vias 3 -> 1
- net Paddle Dah: track 26.0 -> 16.4 mm
- net Paddle_Dit: track 22.4 -> 15.9 mm
Other:
- board text removed: "Dah"
- board text removed: "Dit"
- board text removed: "SK"
