File: KiCad/SignalSlinger/PowerSupply.kicad_sch (KiCad schematic)
At the start: 38 parts, among them J201 Barrel_Jack_Switch, J203 External Fan Power, J204 Controlled Power, U201 LP2985-3.3, U202 LP2985-3.3, U203 TPS63060, U204 TPS22810DBVT

Commit message: Schematic & PCB Updates
o Improvements to DC power routing
Parts:
- added D205: Schottky Diode, Diode_SMD:D_SOD-123, symbol Device:D_Schottky_Filled
- D202: footprint Diode_SMD:D_SMA -> Diode_SMD:D_SMB; Digi-Key Part No. B330A-FDICT-ND -> S3AB-FDICT-ND; LCSC Part Number C110485 -> (none); Link https://www.digikey.com/short/70dw2rqz -> https://www.digikey.com/en/products/detail/diodes-incorpora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; Manufacturer PN B330A-13-F -> S3AB-13-F
- D203, D204: value (none) -> Schottky Diode; footprint (none) -> Diode_SMD:D_SOD-123
Connections:
- net V_ext: now also D205.2 (A); no longer C207.2, D204.1 (K), U203.2 (VIN)
- new net: C207.2, D204.1 (K), D205.1 (K), U203.2 (VIN)
Other:
- moved on the sheet: D204
Changed lines of the file:
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@@
   (title_block
     (title "SignalSlinger")
-    (date "2023-11-21")
-    (rev "2.1")
+    (date "2023-12-10")
+    (rev "2.2")
   )
   (junction (at 187.96 116.84) (diameter 0) (color 0 0 0 0)
   )
-  (junction (at 93.98 33.02) (diameter 0) (color 0 0 0 0)
-  )
   (junction (at 57.15 109.22) (diameter 0) (color 0 0 0 0)
   )
@@
   )
   (junction (at 73.66 33.02) (diameter 0) (color 0 0 0 0)
+  )
+  (junction (at 93.98 46.99) (diameter 0) (color 0 0 0 0)
   )
   (junction (at 100.33 54.61) (diameter 0) (color 0 0 0 0)
@@
     (stroke (width 0) (type default) (color 0 0 0 0))
   )
+  (wire (pts (xy 93.98 46.99) (xy 93.98 54.61))
+    (stroke (width 0) (type default) (color 0 0 0 0))
+  )
   (wire (pts (xy 172.72 68.58) (xy 172.72 64.77))
     (stroke (width 0) (type default) (color 0 0 0 0))
@@
     (stroke (width 0) (type default) (color 0 0 0 0))
   )
+  (wire (pts (xy 93.98 44.45) (xy 93.98 46.99))
+    (stroke (width 0) (type default) (color 0 0 0 0))
+  )
   (wire (pts (xy 156.21 54.61) (xy 163.83 54.61))
     (stroke (width 0) (type default) (color 0 0 0 0))
@@
     (stroke (width 0) (type default) (color 0 0 0 0))
   )
+  (wire (pts (xy 93.98 46.99) (xy 100.33 46.99))
+    (stroke (width 0) (type default) (color 0 0 0 0))
+  )
   (wire (pts (xy 163.83 64.77) (xy 163.83 66.04))
     (stroke (width 0) (type default) (color 0 0 0 0))
@@
     (stroke (width 0) (type default) (color 0 0 0 0))
   )
-  (wire (pts (xy 93.98 33.02) (xy 99.06 33.02))
-    (stroke (width 0) (type default) (color 0 0 0 0))
-  )
   (wire (pts (xy 217.17 41.91) (xy 217.17 60.96))
     (stroke (width 0) (type default) (color 0 0 0 0))
@@
     (stroke (width 0) (type default) (color 0 0 0 0))
   )
-  (wire (pts (xy 93.98 33.02) (xy 93.98 54.61))
+  (wire (pts (xy 93.98 33.02) (xy 93.98 36.83))
     (stroke (width 0) (type default) (color 0 0 0 0))
   )
@@
     (pin "2")
   )
+  (symbol (lib_id "Device:D_Schottky_Filled") (at 93.98 40.64 270) (mirror x) (unit 1)
+    (in_bom yes) (on_board yes) (fields_autoplaced)
+    (property "Reference" "D205" (id 0) (at 96.012 41.3913 90)
+      (effects (font (size 1.27 1.27)) (justify left))
+    )
+    (property "Value" "Schottky Diode" (id 1) (at 91.5471 40.9575 0)
+      (effects (font (size 1.27 1.27)) hide)
+    )
+    (property "Footprint" "Diode_SMD:D_SOD-123" (id 2) (at 93.98 40.64 0)
+      (effects (font (size 1.27 1.27)) hide)
+    )
+    (property "Datasheet" "" (id 3) (at 93.98 40.64 0)
+      (effects (font (size 1.27 1.27)) hide)
+    )
+    (property "Digi-Key Part No." "3757-SS0540_R1_00001CT-ND" (id 4) (at 93.98 40.64 0)
+      (effects (font (size 1.27 1.27)) hide)
+    )
+    (property "Link" "https://www.digikey.com/en/products/detail/panjit-international-inc/SS0540-R1-00001/14660617" (id 5) (at 93.98 40.64 0)
+      (effects (font (size 1.27 1.27)) hide)
+    )
+    (property "Manufacturer" "Panjit International Inc." (id 6) (at 93.98 40.64 0)
+      (effects (font (size 1.27 1.27)) hide)
+    )
+    (property "Manufacturer PN" "SS0540_R1_00001" (id 7) (at 93.98 40.64 0)
+      (effects (font (size 1.27 1.27)) hide)
+    )
+    (property "Description" "DIODE SCHOTTKY 40V 500MA SOD123" (id 8) (at 93.98 40.64 0)
+      (effects (font (size 1.27 1.27)) hide)
+    )
+    (pin "1")
+    (pin "2")
+  )
   (symbol (lib_id "Device:C_Small") (at 87.63 104.14 0) (mirror y) (unit 1)
     (in_bom yes) (on_board yes)
@@
     (pin "2")
   )
-  (symbol (lib_id "Device:D_Schottky_Filled") (at 102.87 33.02 0) (mirror x) (unit 1)
-    (in_bom yes) (on_board yes) (fields_autoplaced)
-    (property "Reference" "D204" (id 0) (at 102.5525 30.5872 0))
-    (property "Value" "" (id 1) (at 102.5525 30.5871 0)
-      (effects (font (size 1.27 1.27)) hide)
-    )
-    (property "Footprint" "" (id 2) (at 102.87 33.02 0)
-      (effects (font (size 1.27 1.27)) hide)
-    )
-    (property "Datasheet" "" (id 3) (at 102.87 33.02 0)
-      (effects (font (size 1.27 1.27)) hide)
-    )
-    (property "Digi-Key Part No." "3757-SS0540_R1_00001CT-ND" (id 4) (at 102.87 33.02 0)
-      (effects (font (size 1.27 1.27)) hide)
-    )
-    (property "Link" "https://www.digikey.com/en/products/detail/panjit-international-inc/SS0540-R1-00001/14660617" (id 5) (at 102.87 33.02 0)
-      (effects (font (size 1.27 1.27)) hide)
-    )
-    (property "Manufacturer" "Panjit International Inc." (id 6) (at 102.87 33.02 0)
-      (effects (font (size 1.27 1.27)) hide)
-    )
-    (property "Manufacturer PN" "SS0540_R1_00001" (id 7) (at 102.87 33.02 0)
-      (effects (font (size 1.27 1.27)) hide)
-    )
-    (property "Description" "DIODE SCHOTTKY 40V 500MA SOD123" (id 8) (at 102.87 33.02 0)
+  (symbol (lib_id "Device:D_Schottky_Filled") (at 104.14 46.99 0) (mirror x) (unit 1)
+    (in_bom yes) (on_board yes) (fields_autoplaced)
+    (property "Reference" "D204" (id 0) (at 103.8225 44.5572 0))
+    (property "Value" "Schottky Diode" (id 1) (at 103.8225 44.5571 0)
+      (effects (font (size 1.27 1.27)) hide)
+    )
+    (property "Footprint" "Diode_SMD:D_SOD-123" (id 2) (at 104.14 46.99 0)
+      (effects (font (size 1.27 1.27)) hide)
+    )
+    (property "Datasheet" "" (id 3) (at 104.14 46.99 0)
+      (effects (font (size 1.27 1.27)) hide)
+    )
+    (property "Digi-Key Part No." "3757-SS0540_R1_00001CT-ND" (id 4) (at 104.14 46.99 0)
+      (effects (font (size 1.27 1.27)) hide)
+    )
+    (property "Link" "https://www.digikey.com/en/products/detail/panjit-international-inc/SS0540-R1-00001/14660617" (id 5) (at 104.14 46.99 0)
+      (effects (font (size 1.27 1.27)) hide)
+    )
+    (property "Manufacturer" "Panjit International Inc." (id 6) (at 104.14 46.99 0)
+      (effects (font (size 1.27 1.27)) hide)
+    )
+    (property "Manufacturer PN" "SS0540_R1_00001" (id 7) (at 104.14 46.99 0)
+      (effects (font (size 1.27 1.27)) hide)
+    )
+    (property "Description" "DIODE SCHOTTKY 40V 500MA SOD123" (id 8) (at 104.14 46.99 0)
       (effects (font (size 1.27 1.27)) hide)
     )
@@
       (effects (font (size 1.27 1.27)) hide)
     )
-    (property "Footprint" "Diode_SMD:D_SMA" (id 2) (at 44.45 33.02 0)
+    (property "Footprint" "Diode_SMD:D_SMB" (id 2) (at 44.45 33.02 0)
       (effects (font (size 1.27 1.27)) hide)
     )
@@
       (effects (font (size 1.27 1.27)) hide)
     )
-    (property "Digi-Key Part No." "B330A-FDICT-ND" (id 4) (at 44.45 33.02 0)
-      (effects (font (size 1.27 1.27)) hide)
-    )
-    (property "Link" "https://www.digikey.com/short/70dw2rqz" (id 5) (at 44.45 33.02 0)
+    (property "Digi-Key Part No." "S3AB-FDICT-ND" (id 4) (at 44.45 33.02 0)
+      (effects (font (size 1.27 1.27)) hide)
+    )
+    (property "Link" "https://www.digikey.com/en/products/detail/diodes-incorporated/S3AB-13-F/814419" (id 5) (at 44.45 33.02 0)
       (effects (font (size 1.27 1.27)) hide)
     )
@@
       (effects (font (size 1.27 1.27)) hide)
     )
-    (property "Manufacturer PN" "B330A-13-F" (id 7) (at 44.45 33.02 0)
-      (effects (font (size 1.27 1.27)) hide)
-    )
-    (property "Description" "DIODE SCHOTTKY 30V 3A SMA" (id 8) (at 44.45 33.02 0)
-      (effects (font (size 1.27 1.27)) hide)
-    )
-    (property "LCSC Part Number" "C110485" (id 9) (at 44.45 33.02 0)
+    (property "Manufacturer PN" "S3AB-13-F" (id 7) (at 44.45 33.02 0)
+      (effects (font (size 1.27 1.27)) hide)
+    )
+    (property "Description" "DIODE GEN PURP 50V 3A SMB" (id 8) (at 44.45 33.02 0)
       (effects (font (size 1.27 1.27)) hide)
     )
@@
     (pin "2")
   )
-  (symbol (lib_id "power:+BATT") (at 106.68 33.02 0) (unit 1)
-    (in_bom yes) (on_board yes) (fields_autoplaced)
-    (property "Reference" "#PWR0218" (id 0) (at 106.68 36.83 0)
-      (effects (font (size 1.27 1.27)) hide)
-    )
-    (property "Value" "+BATT" (id 1) (at 108.077 32.1838 0)
-      (effects (font (size 1.27 1.27)) (justify left))
-    )
-    (property "Footprint" "" (id 2) (at 106.68 33.02 0)
-      (effects (font (size 1.27 1.27)) hide)
-    )
-    (property "Datasheet" "" (id 3) (at 106.68 33.02 0)
+  (symbol (lib_id "power:+BATT") (at 107.95 46.99 0) (unit 1)
+    (in_bom yes) (on_board yes) (fields_autoplaced)
+    (property "Reference" "#PWR0218" (id 0) (at 107.95 50.8 0)
+      (effects (font (size 1.27 1.27)) hide)
+    )
+    (property "Value" "+BATT" (id 1) (at 109.347 46.1538 0)
+      (effects (font (size 1.27 1.27)) (justify left))
+    )
+    (property "Footprint" "" (id 2) (at 107.95 46.99 0)
+      (effects (font (size 1.27 1.27)) hide)
+    )
+    (property "Datasheet" "" (id 3) (at 107.95 46.99 0)
       (effects (font (size 1.27 1.27)) hide)
     )
@@
       (effects (font (size 1.27 1.27)) (justify right))
     )
-    (property "Value" "" (id 1) (at 59.5829 103.1875 0)
-      (effects (font (size 1.27 1.27)) hide)
-    )
-    (property "Footprint" "" (id 2) (at 57.15 102.87 0)
-      (effects (font (size 1.27 1.27)) hide)
-    )
+    (property "Value" "Schottky Diode" (id 1) (at 59.5829 103.1875 0)
+      (effects (font (size 1.27 1.27)) hide)
+    )
+    (property "Footprint" "Diode_SMD:D_SOD-123" (id 2) (at 57.15 102.87 0)
+      (effects (font (size 1.27 1.27)) hide)
+    )

Commit message: Schematic Update
o Power routing improvement
Parts:
- added C217: 330nF, Capacitor_SMD:C_0805_2012Metric, symbol Device:C_Small
- added C218: 100nF, Capacitor_SMD:C_0805_2012Metric, symbol Device:C_Small
- added D206, D207: Schottky Diode, Diode_SMD:D_SOD-123FL, symbol Device:D_Schottky_Filled
- added U205: uA7805, Package_TO_SOT_SMD:SOT-223-4, symbol Regulator_Linear:uA7805
- D203, D204, D205: footprint Diode_SMD:D_SOD-123 -> Diode_SMD:D_SOD-123FL; Digi-Key Part No. 3757-SS0540_R1_00001CT-ND -> RB070MM-30CT-ND; Link https://www.digikey.com/en/products/detail/panjit-internati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 -> https://www.digikey.com/en/products/detail/rohm-semiconduct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; Manufacturer Panjit International Inc. -> Rohm Semiconductor; Manufacturer PN SS0540_R1_00001 -> RB070MM-30TR
Connections:
- net +BATT: no longer D204.2 (A)
- net +VSW: now also D204.2 (A)
- net GND: now also C217.2, C218.2, U205.2 (GND)
- net V+_Charging: now also D206.2 (A); no longer MOD201.4 (Pin_4)
- net V_ext: now also C217.1, U205.1 (IN)
- new net: C218.1, D207.2 (A), U205.3 (OUT)
- new net: D206.1 (K), D207.1 (K), MOD201.4 (Pin_4)
Other:
- moved on the sheet: MOD201
