File: KiCad/SignalSlinger/RF_Filters.kicad_sch (KiCad schematic)
At the start: 13 parts, among them J302 Conn_01x03

Commit message: Updates
o Updated Gerbers
Parts:
- J301: value (none) -> To Antenna; footprint (none) -> Connector_Coaxial:BNC_Amphenol_B6252HB-NPP3G-50_Horizontal
Changed lines of the file:
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@@
   (title_block
     (title "SignalSlinger Design")
-    (date "2023-06-20")
-    (rev "1.0")
+    (date "2023-07-10")
+    (rev "1.1")
   )
   (junction (at 165.1 83.82) (diameter 0) (color 0 0 0 0)
@@
       (effects (font (size 1.27 1.27)) (justify left))
     )
-    (property "Value" "" (id 1) (at 180.3401 85.8154 0)
-      (effects (font (size 1.27 1.27)) (justify left))
-    )
-    (property "Footprint" "" (id 2) (at 177.8 83.82 0)
-      (effects (font (size 1.27 1.27)) hide)
-    )
+    (property "Value" "To Antenna" (id 1) (at 180.3401 85.8154 0)
+      (effects (font (size 1.27 1.27)) (justify left))
+    )
+    (property "Footprint" "Connector_Coaxial:BNC_Amphenol_B6252HB-NPP3G-50_Horizontal" (id 2) (at 177.8 83.82 0)
+      (effects (font (size 1.27 1.27)) hide)
+    )

Commit message: KiCad Updates
Updated Gerbers and schematic
Parts:
- C302, C305: Digi-Key Part No. 399-14552-1-ND -> (none); LCSC Part Number C2327793 -> (none); Link https://www.digikey.com/products/en?keywords=399-14552-1-ND -> (none); Manufacturer PN C0805C112J5GAC7800 -> C325C112KAG5TA
- C303: Digi-Key Part No. 445-5752-1-ND -> (none); LCSC Part Number C2173329 -> (none); Link https://www.digikey.com/products/en?keywords=445-5752-1-ND -> (none); Manufacturer TDK Corporation -> KEMET; Manufacturer PN CGA4F2C0G2A182J085AA -> C325C182JAG5TA
- C304: Digi-Key Part No. 478-10247-1-ND -> (none); LCSC Part Number C2170042 -> (none); Link https://www.digikey.com/products/en?keywords=478-10247-1-ND -> (none); Manufacturer KYOCERA AVX -> KEMET; Manufacturer PN 06031U910FAT2A -> C325C910JAG5TA
Other:
- note added: "L301 & L302: 20T (46 cm) #24 T60-2"
- note removed: "L106 & L108: 20T (46 cm) #24 T60-2 70% Coverage"
Changed lines of the file:
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@@
   )
   (text "40m LPF\n6th order Chebychev\n8MHz 3dB cut-off\nw/ node at 21.5 MHz\n\nL301 & L302 = 1.3uH\nC302 & C305 = 470pF\nC303 = 820pF\nC304 = 43pF"
-    (at 147.32 69.85 0)
+    (at 124.46 125.73 0)
     (effects (font (size 1.27 1.27)) (justify left bottom))
   )
-  (text "L106 & L108:\n20T (46 cm) #24 T60-2 70% Coverage" (at 121.92 97.79 0)
+  (text "L301 & L302:\n20T (46 cm) #24 T60-2 " (at 121.92 97.79 0)
     (effects (font (size 0.9906 0.9906)) (justify left bottom))
   )
@@
     )
     (property "Datasheet" "" (id 3) (at 134.62 88.9 0))
-    (property "Digi-Key Part No." "445-5752-1-ND" (id 4) (at 134.62 88.9 0)
-      (effects (font (size 1.27 1.27)) hide)
-    )
-    (property "Link" "https://www.digikey.com/products/en?keywords=445-5752-1-ND" (id 5) (at 134.62 88.9 0)
-      (effects (font (size 1.524 1.524)) hide)
-    )
-    (property "Manufacturer" "TDK Corporation" (id 6) (at 134.62 88.9 0)
-      (effects (font (size 1.27 1.27)) hide)
-    )
-    (property "Manufacturer PN" "CGA4F2C0G2A182J085AA" (id 7) (at 134.62 88.9 0)
-      (effects (font (size 1.27 1.27)) hide)
-    )
-    (property "Description" "CAP CER 1800PF 100V C0G 0805" (id 8) (at 134.62 88.9 0)
-      (effects (font (size 1.27 1.27)) hide)
-    )
-    (property "LCSC Part Number" "C2173329" (id 9) (at 134.62 88.9 0)
+    (property "Manufacturer" "KEMET" (id 6) (at 134.62 88.9 0)
+      (effects (font (size 1.27 1.27)) hide)
+    )
+    (property "Manufacturer PN" "C325C182JAG5TA" (id 7) (at 134.62 88.9 0)
+      (effects (font (size 1.27 1.27)) hide)
+    )
+    (property "Description" "CAP CER 1800PF 250V C0G 5.08mm" (id 8) (at 134.62 88.9 0)
       (effects (font (size 1.27 1.27)) hide)
     )
@@
     )
     (property "Datasheet" "" (id 3) (at 160.02 88.9 0))
-    (property "Digi-Key Part No." "399-14552-1-ND" (id 4) (at 160.02 88.9 0)
-      (effects (font (size 1.27 1.27)) hide)
-    )
-    (property "Link" "https://www.digikey.com/products/en?keywords=399-14552-1-ND" (id 5) (at 160.02 88.9 0)
-      (effects (font (size 1.524 1.524)) hide)
-    )
     (property "Manufacturer" "KEMET" (id 6) (at 160.02 88.9 0)
       (effects (font (size 1.27 1.27)) hide)
     )
-    (property "Manufacturer PN" "C0805C112J5GAC7800" (id 7) (at 160.02 88.9 0)
-      (effects (font (size 1.27 1.27)) hide)
-    )
-    (property "Description" "CAP CER 1100PF 50V NP0 0805" (id 8) (at 160.02 88.9 0)
-      (effects (font (size 1.27 1.27)) hide)
-    )
-    (property "LCSC Part Number" "C2327793" (id 9) (at 160.02 88.9 0)
-      (effects (font (size 1.27 1.27)) hide)
-    )
-    (pin "1")
-    (pin "2")
-  )
-  (symbol (lib_id "Device:C_Small") (at 116.84 88.9 0) (unit 1)
-    (in_bom yes) (on_board yes)
-    (property "Reference" "C302" (id 0) (at 117.094 87.122 0)
-      (effects (font (size 1.27 1.27)) (justify left))
-    )
-    (property "Value" "1100pF" (id 1) (at 117.094 90.932 0)
-      (effects (font (size 1.27 1.27)) (justify left))
-    )
-    (property "Footprint" "Capacitor_THT:C_Rect_L7.0mm_W2.5mm_P5.00mm" (id 2) (at 116.84 88.9 0)
-      (effects (font (size 1.27 1.27)) hide)
-    )
-    (property "Datasheet" "" (id 3) (at 116.84 88.9 0))
-    (property "Digi-Key Part No." "399-14552-1-ND" (id 4) (at 116.84 88.9 0)
-      (effects (font (size 1.27 1.27)) hide)
-    )
-    (property "Link" "https://www.digikey.com/products/en?keywords=399-14552-1-ND" (id 5) (at 116.84 88.9 0)
-      (effects (font (size 1.524 1.524)) hide)
-    )
-    (property "Manufacturer" "KEMET" (id 6) (at 116.84 88.9 0)
-      (effects (font (size 1.27 1.27)) hide)
-    )
-    (property "Manufacturer PN" "C0805C112J5GAC7800" (id 7) (at 116.84 88.9 0)
-      (effects (font (size 1.27 1.27)) hide)
-    )
-    (property "Description" "CAP CER 1100PF 50V NP0 0805" (id 8) (at 116.84 88.9 0)
-      (effects (font (size 1.27 1.27)) hide)
-    )
-    (property "LCSC Part Number" "C2327793" (id 9) (at 116.84 88.9 0)
+    (property "Manufacturer PN" "C325C112KAG5TA" (id 7) (at 160.02 88.9 0)
+      (effects (font (size 1.27 1.27)) hide)
+    )
+    (property "Description" "CAP CER 1100PF 250V NP0 5.08mm" (id 8) (at 160.02 88.9 0)
       (effects (font (size 1.27 1.27)) hide)
     )
@@
     )
     (property "Datasheet" "" (id 3) (at 151.13 76.2 0))
-    (property "Digi-Key Part No." "478-10247-1-ND" (id 4) (at 151.13 76.2 0)
-      (effects (font (size 1.27 1.27)) hide)
-    )
-    (property "Link" "https://www.digikey.com/products/en?keywords=478-10247-1-ND" (id 5) (at 151.13 76.2 0)
-      (effects (font (size 1.524 1.524)) hide)
-    )
-    (property "Manufacturer" "KYOCERA AVX" (id 6) (at 151.13 76.2 90)
-      (effects (font (size 1.27 1.27)) hide)
-    )
-    (property "Manufacturer PN" "06031U910FAT2A" (id 7) (at 151.13 76.2 90)
-      (effects (font (size 1.27 1.27)) hide)
-    )
-    (property "Description" "CAP CER 91PF 100V NP0 0603" (id 8) (at 151.13 76.2 90)
-      (effects (font (size 1.27 1.27)) hide)
-    )
-    (property "LCSC Part Number" "C2170042" (id 9) (at 151.13 76.2 0)
+    (property "Manufacturer" "KEMET" (id 6) (at 151.13 76.2 90)
+      (effects (font (size 1.27 1.27)) hide)
+    )
+    (property "Manufacturer PN" "C325C910JAG5TA" (id 7) (at 151.13 76.2 90)
+      (effects (font (size 1.27 1.27)) hide)
+    )
+    (property "Description" "CAP CER 91PF 250V NP0 5.08mm" (id 8) (at 151.13 76.2 90)
       (effects (font (size 1.27 1.27)) hide)
     )
@@
     (pin "1")
   )
+  (symbol (lib_id "Device:C_Small") (at 116.84 88.9 0) (unit 1)
+    (in_bom yes) (on_board yes)
+    (property "Reference" "C302" (id 0) (at 117.094 87.122 0)
+      (effects (font (size 1.27 1.27)) (justify left))
+    )
+    (property "Value" "1100pF" (id 1) (at 117.094 90.932 0)
+      (effects (font (size 1.27 1.27)) (justify left))
+    )
+    (property "Footprint" "Capacitor_THT:C_Rect_L7.0mm_W2.5mm_P5.00mm" (id 2) (at 116.84 88.9 0)
+      (effects (font (size 1.27 1.27)) hide)
+    )
+    (property "Datasheet" "" (id 3) (at 116.84 88.9 0))
+    (property "Manufacturer" "KEMET" (id 6) (at 116.84 88.9 0)
+      (effects (font (size 1.27 1.27)) hide)
+    )
+    (property "Manufacturer PN" "C325C112KAG5TA" (id 7) (at 116.84 88.9 0)
+      (effects (font (size 1.27 1.27)) hide)
+    )
+    (property "Description" "CAP CER 1100PF 250V NP0 5.08mm" (id 8) (at 116.84 88.9 0)
+      (effects (font (size 1.27 1.27)) hide)
+    )
+    (pin "1")
+    (pin "2")
+  )
   (symbol (lib_id "power:GND") (at 119.38 80.01 0) (unit 1)

Commit message: Schematic Updates
o Added support for a linear adjustable voltage regulator
o Added a switch
o Re-arranged components for a better fit
Parts:
- removed J302: Conn_01x03, Connector_PinHeader_2.54mm:PinHeader_1x03_P2.54mm_Vertical, symbol Connector_Generic:Conn_01x03
- removed JP301: QRP disable, Jumper:SolderJumper-2_P1.3mm_Bridged_RoundedPad1.0x1.5mm, symbol Jumper:SolderJumper_2_Bridged
Connections:
- net RF_Raw: now also C301.1
- no-connect marks 1 -> 0
Other:
- note removed: "To QRPP Board"
Changed lines of the file:
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@@
   (junction (at 143.51 83.82) (diameter 0) (color 0 0 0 0)
   )
-  (junction (at 95.25 86.36) (diameter 0) (color 0 0 0 0)
-  )
   (junction (at 116.84 83.82) (diameter 0) (color 0 0 0 0)
   )
-  (junction (at 102.87 83.82) (diameter 0) (color 0 0 0 0)
-  )
   (junction (at 160.02 83.82) (diameter 0) (color 0 0 0 0)
   )
-  (no_connect (at 95.25 81.28))
-  (wire (pts (xy 95.25 91.44) (xy 95.25 86.36))
-    (stroke (width 0) (type default) (color 0 0 0 0))
-  )
   (wire (pts (xy 116.84 83.82) (xy 116.84 86.36))
     (stroke (width 0) (type default) (color 0 0 0 0))
   )
-  (wire (pts (xy 95.25 83.82) (xy 102.87 83.82))
-    (stroke (width 0) (type default) (color 0 0 0 0))
-  )
   (wire (pts (xy 143.51 83.82) (xy 144.78 83.82))
     (stroke (width 0) (type default) (color 0 0 0 0))
@@
     (stroke (width 0) (type default) (color 0 0 0 0))
   )
-  (wire (pts (xy 91.44 91.44) (xy 95.25 91.44))
-    (stroke (width 0) (type default) (color 0 0 0 0))
-  )
   (wire (pts (xy 102.87 83.82) (xy 106.68 83.82))
     (stroke (width 0) (type default) (color 0 0 0 0))
@@
   )
   (wire (pts (xy 160.02 76.2) (xy 160.02 83.82))
-    (stroke (width 0) (type default) (color 0 0 0 0))
-  )
-  (wire (pts (xy 102.87 83.82) (xy 102.87 86.36))
     (stroke (width 0) (type default) (color 0 0 0 0))
   )
@@
     (effects (font (size 0.9906 0.9906)) (justify left bottom))
   )
-  (text "To QRPP Board" (at 71.12 83.82 0)
-    (effects (font (size 1.27 1.27)) (justify left bottom))
-  )
   (text "80m LPF" (at 129.54 63.5 0)
     (effects (font (size 2.0066 2.0066) (thickness 0.4013) bold) (justify left bottom))
   )
-  (global_label "RF_Raw" (shape input) (at 91.44 91.44 180) (fields_autoplaced)
+  (global_label "RF_Raw" (shape input) (at 102.87 83.82 180) (fields_autoplaced)
     (effects (font (size 1 1)) (justify right))
-    (property "Intersheet References" "${INTERSHEET_REFS}" (id 0) (at 83.9686 91.3775 0)
+    (property "Intersheet References" "${INTERSHEET_REFS}" (id 0) (at 95.3986 83.7575 0)
       (effects (font (size 1 1)) (justify right) hide)
     )
@@
     (pin "2")
   )
-  (symbol (lib_id "Jumper:SolderJumper_2_Bridged") (at 99.06 86.36 0) (unit 1)
-    (in_bom yes) (on_board yes)
-    (property "Reference" "JP301" (id 0) (at 99.06 88.9 0))
-    (property "Value" "QRP disable" (id 1) (at 102.87 91.44 0))
-    (property "Footprint" "Jumper:SolderJumper-2_P1.3mm_Bridged_RoundedPad1.0x1.5mm" (id 2) (at 99.06 86.36 0)
-      (effects (font (size 1.27 1.27)) hide)
-    )
-    (property "Datasheet" "~" (id 3) (at 99.06 86.36 0)
-      (effects (font (size 1.27 1.27)) hide)
-    )
-    (pin "1")
-    (pin "2")
-  )
   (symbol (lib_id "Device:C_Small") (at 109.22 83.82 90) (unit 1)
     (in_bom yes) (on_board yes)
@@
     (pin "1")
   )
-  (symbol (lib_id "Connector_Generic:Conn_01x03") (at 90.17 83.82 180) (unit 1)
-    (in_bom yes) (on_board yes)
-    (property "Reference" "J302" (id 0) (at 87.63 86.36 90)
-      (effects (font (size 1.27 1.27)) (justify right))
-    )
-    (property "Value" "Conn_01x03" (id 1) (at 91.8722 79.248 90)
-      (effects (font (size 1.27 1.27)) (justify right) hide)
-    )
-    (property "Footprint" "Connector_PinHeader_2.54mm:PinHeader_1x03_P2.54mm_Vertical" (id 2) (at 90.17 83.82 0)
-      (effects (font (size 1.27 1.27)) hide)
-    )
-    (property "Datasheet" "~" (id 3) (at 90.17 83.82 0)
-      (effects (font (size 1.27 1.27)) hide)
-    )
-    (pin "1")
-    (pin "2")
-    (pin "3")
-  )
   (symbol (lib_id "Connector:TEST_SCOPE") (at 116.84 80.01 0) (unit 1)

Commit message: Updated Schematic Rev
Rev 1.2
Other:
- title: SignalSlinger Design -> SignalSlinger
Changed lines of the file:
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@@
   (paper "A4")
   (title_block
-    (title "SignalSlinger Design")
-    (date "2023-07-10")
-    (rev "1.1")
+    (title "SignalSlinger")
+    (date "2023-11-17")
+    (rev "1.2")
   )
   (junction (at 165.1 83.82) (diameter 0) (color 0 0 0 0)

Commit message: Rev 2.3
Updates from initial PCB build.
Added thermal fuse F101
Support for regulated voltage
Support for charging LiPo via transmitter external power source
Updated BOM
Updated PCB and schematic
Parts:
- C302, C305: footprint Capacitor_THT:C_Rect_L7.0mm_W2.5mm_P5.00mm -> Capacitor_SMD:C_0805_2012Metric; Manufacturer KEMET -> Murata Electronics; Manufacturer PN C325C112KAG5TA -> GRM2195C2A112JA01D
- C303: footprint Capacitor_THT:C_Rect_L7.0mm_W2.5mm_P5.00mm -> Capacitor_SMD:C_0805_2012Metric; Manufacturer KEMET -> Murata Electronics; Manufacturer PN C325C182JAG5TA -> GCM2165C2A182GA16D
- C304: footprint Capacitor_THT:C_Rect_L7.0mm_W2.5mm_P5.00mm -> Capacitor_SMD:C_0805_2012Metric; Manufacturer KEMET -> KYOCERA AVX; Manufacturer PN C325C910JAG5TA -> 08051A910FAT2A
Changed lines of the file:
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@@
   (title_block
     (title "SignalSlinger")
-    (date "2023-12-10")
-    (rev "2.2")
+    (date "2024-04-13")
+    (rev "2.3")
   )
   (junction (at 165.1 83.82) (diameter 0) (color 0 0 0 0)
@@
       (effects (font (size 1.27 1.27)) (justify left))
     )
-    (property "Footprint" "Capacitor_THT:C_Rect_L7.0mm_W2.5mm_P5.00mm" (id 2) (at 134.62 88.9 0)
+    (property "Footprint" "Capacitor_SMD:C_0805_2012Metric" (id 2) (at 134.62 88.9 0)
       (effects (font (size 1.27 1.27)) hide)
     )
     (property "Datasheet" "" (id 3) (at 134.62 88.9 0))
-    (property "Manufacturer" "KEMET" (id 6) (at 134.62 88.9 0)
-      (effects (font (size 1.27 1.27)) hide)
-    )
-    (property "Manufacturer PN" "C325C182JAG5TA" (id 7) (at 134.62 88.9 0)
-      (effects (font (size 1.27 1.27)) hide)
-    )
-    (property "Description" "CAP CER 1800PF 250V C0G 5.08mm" (id 8) (at 134.62 88.9 0)
-      (effects (font (size 1.27 1.27)) hide)
-    )
-    (pin "1")
-    (pin "2")
-  )
-  (symbol (lib_id "Device:C_Small") (at 160.02 88.9 0) (unit 1)
-    (in_bom yes) (on_board yes)
-    (property "Reference" "C305" (id 0) (at 160.274 87.122 0)
-      (effects (font (size 1.27 1.27)) (justify left))
-    )
-    (property "Value" "1100pF" (id 1) (at 160.274 90.932 0)
-      (effects (font (size 1.27 1.27)) (justify left))
-    )
-    (property "Footprint" "Capacitor_THT:C_Rect_L7.0mm_W2.5mm_P5.00mm" (id 2) (at 160.02 88.9 0)
-      (effects (font (size 1.27 1.27)) hide)
-    )
-    (property "Datasheet" "" (id 3) (at 160.02 88.9 0))
-    (property "Manufacturer" "KEMET" (id 6) (at 160.02 88.9 0)
-      (effects (font (size 1.27 1.27)) hide)
-    )
-    (property "Manufacturer PN" "C325C112KAG5TA" (id 7) (at 160.02 88.9 0)
-      (effects (font (size 1.27 1.27)) hide)
-    )
-    (property "Description" "CAP CER 1100PF 250V NP0 5.08mm" (id 8) (at 160.02 88.9 0)
+    (property "Manufacturer" "Murata Electronics" (id 6) (at 134.62 88.9 0)
+      (effects (font (size 1.27 1.27)) hide)
+    )
+    (property "Manufacturer PN" "GCM2165C2A182GA16D" (id 7) (at 134.62 88.9 0)
+      (effects (font (size 1.27 1.27)) hide)
+    )
+    (property "Description" "Multilayer Ceramic Capacitors MLCC - SMD/SMT 1800 pF 100 VDC 2% 0805 C0G (NP0) AEC-Q200" (id 8) (at 134.62 88.9 0)
       (effects (font (size 1.27 1.27)) hide)
     )
@@
       (effects (font (size 1.27 1.27)) (justify left))
     )
-    (property "Footprint" "Capacitor_THT:C_Rect_L7.0mm_W2.5mm_P5.00mm" (id 2) (at 151.13 76.2 0)
+    (property "Footprint" "Capacitor_SMD:C_0805_2012Metric" (id 2) (at 151.13 76.2 0)
       (effects (font (size 1.27 1.27)) hide)
     )
     (property "Datasheet" "" (id 3) (at 151.13 76.2 0))
-    (property "Manufacturer" "KEMET" (id 6) (at 151.13 76.2 90)
-      (effects (font (size 1.27 1.27)) hide)
-    )
-    (property "Manufacturer PN" "C325C910JAG5TA" (id 7) (at 151.13 76.2 90)
-      (effects (font (size 1.27 1.27)) hide)
-    )
-    (property "Description" "CAP CER 91PF 250V NP0 5.08mm" (id 8) (at 151.13 76.2 90)
+    (property "Manufacturer" "KYOCERA AVX" (id 6) (at 151.13 76.2 90)
+      (effects (font (size 1.27 1.27)) hide)
+    )
+    (property "Manufacturer PN" "08051A910FAT2A" (id 7) (at 151.13 76.2 90)
+      (effects (font (size 1.27 1.27)) hide)
+    )
+    (property "Description" "Multilayer Ceramic Capacitors MLCC - SMD/SMT 100V 91pF C0G 0805 1%" (id 8) (at 151.13 76.2 90)
+      (effects (font (size 1.27 1.27)) hide)
+    )
+    (pin "1")
+    (pin "2")
+  )
+  (symbol (lib_id "Device:C_Small") (at 160.02 88.9 0) (unit 1)
+    (in_bom yes) (on_board yes)
+    (property "Reference" "C305" (id 0) (at 160.274 87.122 0)
+      (effects (font (size 1.27 1.27)) (justify left))
+    )
+    (property "Value" "1100pF" (id 1) (at 160.274 90.932 0)
+      (effects (font (size 1.27 1.27)) (justify left))
+    )
+    (property "Footprint" "Capacitor_SMD:C_0805_2012Metric" (id 2) (at 160.02 88.9 0)
+      (effects (font (size 1.27 1.27)) hide)
+    )
+    (property "Datasheet" "" (id 3) (at 160.02 88.9 0))
+    (property "Manufacturer" "Murata Electronics" (id 6) (at 160.02 88.9 0)
+      (effects (font (size 1.27 1.27)) hide)
+    )
+    (property "Manufacturer PN" "GRM2195C2A112JA01D" (id 7) (at 160.02 88.9 0)
+      (effects (font (size 1.27 1.27)) hide)
+    )
+    (property "Description" "Multilayer Ceramic Capacitors MLCC - SMD/SMT 1100 pF 100 VDC 5% 0805 C0G (NP0)" (id 8) (at 160.02 88.9 0)
       (effects (font (size 1.27 1.27)) hide)
     )
@@
       (effects (font (size 1.27 1.27)) (justify left))
     )
-    (property "Footprint" "Capacitor_THT:C_Rect_L7.0mm_W2.5mm_P5.00mm" (id 2) (at 116.84 88.9 0)
+    (property "Footprint" "Capacitor_SMD:C_0805_2012Metric" (id 2) (at 116.84 88.9 0)
       (effects (font (size 1.27 1.27)) hide)
     )
     (property "Datasheet" "" (id 3) (at 116.84 88.9 0))
-    (property "Manufacturer" "KEMET" (id 6) (at 116.84 88.9 0)
-      (effects (font (size 1.27 1.27)) hide)
-    )
-    (property "Manufacturer PN" "C325C112KAG5TA" (id 7) (at 116.84 88.9 0)
-      (effects (font (size 1.27 1.27)) hide)
-    )
-    (property "Description" "CAP CER 1100PF 250V NP0 5.08mm" (id 8) (at 116.84 88.9 0)
-      (effects (font (size 1.27 1.27)) hide)
-    )
+    (property "Manufacturer" "Murata Electronics" (id 6) (at 116.84 88.9 0)
+      (effects (font (size 1.27 1.27)) hide)
+    )
+    (property "Manufacturer PN" "GRM2195C2A112JA01D" (id 7) (at 116.84 88.9 0)
+      (effects (font (size 1.27 1.27)) hide)
+    )
+    (property "Description" "Multilayer Ceramic Capacitors MLCC - SMD/SMT 1100 pF 100 VDC 5% 0805 C0G (NP0)" (id 8) (at 116.84 88.9 0)
+      (effects (font (size 1.27 1.27)) hide)
+    )
