File: KiCad/SignalSlinger/RF_Filters.kicad_sch (KiCad schematic)
At the start: 11 parts, among them J301 To Antenna

Commit message: Added voltage divider
Now supports monitoring external battery voltage.
Parts:
- L301, L302: footprint Inductors:Toroid_T-60_2TH -> Inductors:Toroid_T-60_2TH_Vertical
Changed lines of the file:
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@@
     (title "SignalSlinger")
     (date "2024-04-15")
-    (rev "2.4")
+    (rev "3.0")
   )
   (junction (at 165.1 83.82) (diameter 0) (color 0 0 0 0)
@@
     (property "Reference" "L302" (id 0) (at 151.13 81.28 0))
     (property "Value" "2.7uH" (id 1) (at 151.13 85.09 0))
-    (property "Footprint" "Inductors:Toroid_T-60_2TH" (id 2) (at 151.13 83.82 0)
+    (property "Footprint" "Inductors:Toroid_T-60_2TH_Vertical" (id 2) (at 151.13 83.82 0)
       (effects (font (size 1.27 1.27)) hide)
     )
@@
     (property "Reference" "L301" (id 0) (at 125.73 81.28 0))
     (property "Value" "2.7uH" (id 1) (at 125.73 85.09 0))
-    (property "Footprint" "Inductors:Toroid_T-60_2TH" (id 2) (at 125.73 83.82 0)
+    (property "Footprint" "Inductors:Toroid_T-60_2TH_Vertical" (id 2) (at 125.73 83.82 0)
       (effects (font (size 1.27 1.27)) hide)
     )
